File: NordBoard/NordBoard.kicad_pcb (KiCad board)
At the start: 2 copper layers, 276 x 89.5 mm, 93 parts, among them SW1 SW_Push, SW10 SW_Push, SW11 SW_Push, SW12 SW_Push, SW13 SW_Push, SW14 SW_Push, SW15 SW_Push, SW16 SW_Push, SW17 SW_Push, SW18 SW_Push, SW19 SW_Push, SW2 SW_Push, SW20 SW_Push, SW21 SW_Push, SW22 SW_Push, SW23 SW_Push, SW24 SW_Push, SW25 SW_Push, SW26 SW_Push, SW27 SW_Push, SW28 SW_Push, SW29 SW_Push, SW3 SW_Push, SW30 SW_Push, SW31 SW_Push, SW32 SW_Push, SW33 SW_Push, SW34 SW_Push, SW35 SW_Push, SW36 SW_Push, SW37 SW_Push, SW38 SW_Push, SW39 SW_Push, SW4 SW_Push, SW40 SW_Push, SW5 SW_Push, SW6 SW_Push, SW7 SW_Push, SW8 SW_Push, SW9 SW_Push, U1 XIAO-RP2040-DIP, U2 XIAO-RP2040-DIP

Commit message: chore: pcb board cleanup
Parts:
- removed H7, H8: MountingHole, MountingHole:MountingHole_2.2mm_M2
- moved H6 117.5 mm to (252.5, 24.0)
- moved H4 85.2 mm to (159.5, 75.0)
- moved H5 69.4 mm to (210.0, 90.0)
- moved H2 5.15 mm to (90.0, 90.0)
Other:
- outline, holes or cut-outs redrawn

Commit message: feat: implement mousebites
Parts:
- added B4: MouseBite, PCM_marbastlib-various:mousebites_2mm, F.Cu at (148.5, 85.9)
- added B5: MouseBite, PCM_marbastlib-various:mousebites_2mm, F.Cu at (148.4, 98.0)
- B1, B2, B3: footprint Panelization:mouse-bite-5mm-slot -> PCM_marbastlib-various:mousebites_2mm
- moved B3 17.9 mm to (148.5, 73.9), turned to 180 degrees
- moved B2 4.75 mm to (148.4, 50.0), turned to 180 degrees
- moved B1 2.86 mm to (148.5, 61.9), turned to 180 degrees
- moved D1 2.50 mm to (23.0, 47.5)
- moved D10 2.50 mm to (80.0, 34.0)
- moved D11 2.50 mm to (80.0, 53.0)
- moved D12 2.50 mm to (80.0, 72.0)
- moved D13 2.50 mm to (99.0, 37.0)
- moved D14 2.50 mm to (99.0, 56.0)
- moved D15 2.50 mm to (99.0, 75.0)
- moved D16 2.50 mm to (118.1, 99.5)
- moved D17 2.50 mm to (118.0, 41.4)
- moved D18 2.50 mm to (118.0, 60.4)
- moved D19 2.50 mm to (118.0, 79.5)
- moved D2 2.50 mm to (23.0, 66.5)
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Other:
- board size 276 x 89.5 mm -> 273 x 89.5 mm

Commit message: feat: finish PCB awaiting peer review + silkscreen
Parts:
- moved B5 46.5 mm to (147.5, 144.5)
- moved B4 45.3 mm to (147.5, 131.1)
- moved H5 45.3 mm to (197.0, 133.5)
- moved H2 44.1 mm to (100.0, 133.5)
- moved D27 43.5 mm to (218.0, 77.3)
- moved D28 43.5 mm to (218.0, 96.3)
- moved D29 43.5 mm to (218.0, 115.3)
- moved D33 43.5 mm to (256.1, 90.3)
- moved D34 43.5 mm to (256.1, 109.3)
- moved D35 43.5 mm to (256.1, 128.3)
- moved D38 43.5 mm to (275.1, 110.0)
- moved D39 43.5 mm to (274.9, 129.2)
- moved SW15 43.5 mm to (98.0, 109.1)
- moved SW28 43.5 mm to (218.0, 86.8)
- moved SW29 43.5 mm to (218.0, 105.8)
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Other:
- outline, holes or cut-outs redrawn
- board text added: "Alec with a heart"
- board text added: "Eggdog"
- board text added: "Hack club logo"
- board text added: "NordBoard"
- board text added: "Permafrost logo here"

Commit message: feat: finish PCB silkscreen, export STEP
Other:
- board text added: "1"
- board text removed: "Alec with a heart"
- board text removed: "Eggdog"
- board text removed: "Hack club logo"
- board text removed: "Permafrost logo here"

Commit message: fix: fix pcb errors
Connections:
- U1 pad 13: GND -> unconnected-(U1-GND-Pad13)
- U2 pad 13: GND -> unconnected-(U2-GND-Pad13)
Changed lines of the file:
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@@
 	(net 64 "unconnected-(U1-VBUS-Pad14)")
 	(net 65 "unconnected-(U1-3V3-Pad12)_1")
-	(net 66 "GND")
+	(net 66 "unconnected-(U1-GND-Pad13)")
 	(net 67 "unconnected-(U1-VBUS-Pad14)_1")
 	(net 68 "unconnected-(U2-VBUS-Pad14)")
@@
 	(net 72 "unconnected-(U2-VBUS-Pad14)_1")
 	(net 73 "unconnected-(U2-3V3-Pad12)_1")
+	(net 74 "unconnected-(U1-GND-Pad13)_1")
+	(net 75 "unconnected-(U2-GND-Pad13)")
+	(net 76 "unconnected-(U2-GND-Pad13)_1")
 	(footprint "PCM_marbastlib-choc:SW_choc_v1_1u"
 		(layer "F.Cu")
@@
 			(layers "*.Cu" "*.Mask")
 			(remove_unused_layers no)
-			(net 66 "GND")
+			(net 74 "unconnected-(U1-GND-Pad13)_1")
 			(pinfunction "GND")
-			(pintype "passive")
+			(pintype "passive+no_connect")
 		)
 		(pad "13" smd roundrect
@@
 			(layers "F.Cu" "F.Mask")
 			(roundrect_rratio 0.1)
-			(net 66 "GND")
+			(net 66 "unconnected-(U1-GND-Pad13)")
 			(pinfunction "GND")
-			(pintype "passive")
+			(pintype "passive+no_connect")
 			(thermal_bridge_angle 45)
 		)
@@
 			(layers "*.Cu" "*.Mask")
 			(remove_unused_layers no)
-			(net 66 "GND")
+			(net 76 "unconnected-(U2-GND-Pad13)_1")
 			(pinfunction "GND")
-			(pintype "passive")
+			(pintype "passive+no_connect")
 		)
 		(pad "13" smd roundrect
@@
 			(layers "F.Cu" "F.Mask")
 			(roundrect_rratio 0.1)
-			(net 66 "GND")
+			(net 75 "unconnected-(U2-GND-Pad13)")
 			(pinfunction "GND")
-			(pintype "passive")
+			(pintype "passive+no_connect")
 			(thermal_bridge_angle 45)
 		)
