File: NordBoard/NordBoard.kicad_sch (KiCad schematic)
At the start: 5 parts

Commit message: journal and some work
Parts:
- added D1, D10, D11, D12, D13, D14, D15, D16, D17, D18, D19, D2, D20, D21, D22, D23, D24, D25, D26, D27, D28, D29, D3, D30, D31, D32, D33, D34, D35, D36, D37, D38, D39, D4, D40, D41, D42, D5, D6, D7, D8, D9: D, Diode_SMD:D_SMA-SMB_Universal_Handsoldering, symbol Device:D
- added H1, H2, H3, H4, H5, H6: MountingHole, MountingHole:MountingHole_2.2mm_M2, symbol Mechanical:MountingHole
- added SW1, SW10, SW11, SW12, SW13, SW14, SW15, SW16, SW17, SW18, SW19, SW2, SW20, SW21, SW22, SW23, SW24, SW25, SW26, SW27, SW28, SW29, SW3, SW30, SW31, SW32, SW33, SW34, SW35, SW36, SW37, SW38, SW39, SW4, SW40, SW41, SW42, SW5, SW6, SW7, SW8, SW9: SW_Push, PCM_marbastlib-choc:SW_choc_v1_1u, symbol Switch:SW_Push
- added U1, U2: XIAO-RP2040-DIP, Seeed Studio XIAO Series Library:XIAO-RP2040-DIP, symbol Seeed_Studio_XIAO_Series:XIAO-RP2040-DIP
Connections:
- new net: D25.2 (A), SW25.2
- new net: D15.2 (A), SW15.2
- new net: D2.2 (A), SW2.2
- new net: D11.2 (A), SW11.2
- new net: D14.2 (A), SW14.2
- new net: D9.2 (A), SW9.2
- new net: D19.2 (A), SW19.2
- new net: D20.2 (A), SW20.2
- new net: D18.2 (A), SW18.2
- new net: D39.2 (A), SW39.2
- new net: D10.2 (A), SW10.2
- new net: D16.2 (A), SW16.2
- new net: D6.2 (A), SW6.2
- new net: D34.2 (A), SW34.2
- new net: D5.2 (A), SW5.2
- new net: D28.2 (A), SW28.2
- new net: D24.2 (A), SW24.2
- new net: D21.2 (A), SW21.2
- new net: D12.2 (A), SW12.2
- new net: D7.2 (A), SW7.2
- new net: D29.2 (A), SW29.2
- new net: D38.2 (A), SW38.2
- new net: D23.2 (A), SW23.2
- new net: D26.2 (A), SW26.2
- new net: D40.2 (A), SW40.2
- new net: D35.2 (A), SW35.2
- new net: D36.2 (A), SW36.2
- new net: D30.2 (A), SW30.2
- new net: D27.2 (A), SW27.2
- new net: D42.2 (A), SW42.2
- new net: D22.2 (A), SW22.2
- new net: D17.2 (A), SW17.2
- new net: D8.2 (A), SW8.2
- new net: D1.2 (A), SW1.2
- new net: D33.2 (A), SW33.2
- new net: D31.2 (A), SW31.2
- new net: D37.2 (A), SW37.2
- new net: D3.2 (A), SW3.2
- new net: D13.2 (A), SW13.2
- new net: D32.2 (A), SW32.2
- new net: D41.2 (A), SW41.2
- new net: D4.2 (A), SW4.2
- new net COL0: SW1.1, SW2.1, SW22.1, SW23.1, SW24.1, SW25.1, SW3.1, SW4.1, U1.2 (GPIO27/ADC1/A1), U2.2 (GPIO27/ADC1/A1)
- new net COL1: SW26.1, SW27.1, SW28.1, SW5.1, SW6.1, SW7.1, U1.3 (GPIO28/ADC2/A2), U2.3 (GPIO28/ADC2/A2)
- new net COL2: SW10.1, SW29.1, SW30.1, SW31.1, SW8.1, SW9.1, U1.4 (GPIO29/ADC3/A3), U2.4 (GPIO29/ADC3/A3)
- new net COL3: SW11.1, SW12.1, SW13.1, SW32.1, SW33.1, SW34.1, U1.5 (GPIO6/SDA), U2.5 (GPIO6/SDA)
- new net COL4: SW14.1, SW15.1, SW16.1, SW17.1, SW35.1, SW36.1, SW37.1, SW38.1, U1.6 (GPIO7/SCL), U2.6 (GPIO7/SCL)
- new net COL5: SW18.1, SW19.1, SW20.1, SW21.1, SW39.1, SW40.1, SW41.1, SW42.1, U1.7 (GPIO0/TX), U2.7 (GPIO0/TX)
- new net ROW0: D1.1 (K), D11.1 (K), D14.1 (K), D18.1 (K), D22.1 (K), D26.1 (K), D29.1 (K), D32.1 (K), D35.1 (K), D39.1 (K), D5.1 (K), D8.1 (K), U1.11 (GPIO3/MOSI), U2.11 (GPIO3/MOSI)
- new net ROW1: D12.1 (K), D15.1 (K), D19.1 (K), D2.1 (K), D23.1 (K), D27.1 (K), D30.1 (K), D33.1 (K), D36.1 (K), D40.1 (K), D6.1 (K), D9.1 (K), U1.10 (GPIO4/MISO), U2.10 (GPIO4/MISO)
- new net ROW2: D10.1 (K), D13.1 (K), D16.1 (K), D20.1 (K), D24.1 (K), D28.1 (K), D3.1 (K), D31.1 (K), D34.1 (K), D37.1 (K), D41.1 (K), D7.1 (K), U1.9 (GPIO2/SCK), U2.9 (GPIO2/SCK)
- new net ROW3: D17.1 (K), D21.1 (K), D25.1 (K), D38.1 (K), D4.1 (K), D42.1 (K), U1.8 (GPIO1/RX), U2.8 (GPIO1/RX)
- no-connect marks 0 -> 8
Other:
- removed sheet left
- removed sheet right
- note added: "Left Matrix"
- note added: "Left Mounting"
- note added: "Left Xiao"
- note added: "Right Matrix"
- note added: "Right Mounting"
- note added: "Right Xiao"
- moved on the sheet: B1, B2, B3, B4, B5
