File: NordBoard.kicad_pcb (KiCad board)
At the start: 2 copper layers, 273 x 89.5 mm, 93 parts, among them SW1 SW_Push, SW10 SW_Push, SW11 SW_Push, SW12 SW_Push, SW13 SW_Push, SW14 SW_Push, SW15 SW_Push, SW16 SW_Push, SW17 SW_Push, SW18 SW_Push, SW19 SW_Push, SW2 SW_Push, SW20 SW_Push, SW21 SW_Push, SW22 SW_Push, SW23 SW_Push, SW24 SW_Push, SW25 SW_Push, SW26 SW_Push, SW27 SW_Push, SW28 SW_Push, SW29 SW_Push, SW3 SW_Push, SW30 SW_Push, SW31 SW_Push, SW32 SW_Push, SW33 SW_Push, SW34 SW_Push, SW35 SW_Push, SW36 SW_Push, SW37 SW_Push, SW38 SW_Push, SW39 SW_Push, SW4 SW_Push, SW40 SW_Push, SW5 SW_Push, SW6 SW_Push, SW7 SW_Push, SW8 SW_Push, SW9 SW_Push, U1 XIAO-RP2040-DIP, U2 XIAO-RP2040-DIP

Commit message: major feat: completely restructure project, new switches, no more path hardcoding
Parts:
- added D50: D, Diode_SMD:D_SMA-SMB_Universal_Handsoldering, F.Cu at (22.5, 148.0)
- added D51: D, Diode_SMD:D_SMA-SMB_Universal_Handsoldering, F.Cu at (275.1, 148.5)
- added SW50: SW_Push, PCM_marbastlib-choc:SW_choc_v1_1u, F.Cu at (22.0, 138.5)
- added SW51: SW_Push, PCM_marbastlib-choc:SW_choc_v1_1u, F.Cu at (275.0, 139.0)
- U1, U2: footprint Seeed Studio XIAO Series Library:XIAO-RP2040-DIP -> kicad_care_package:XIAO-RP2040-DIP
Connections:
- D1 pad 1: /left/ROW0 -> /ROW0
- D10 pad 1: /left/ROW0 -> /ROW0
- D11 pad 1: /left/ROW1 -> /ROW1
- D12 pad 1: /left/ROW2 -> /ROW2
- D13 pad 1: /left/ROW0 -> /ROW0
- D14 pad 1: /left/ROW1 -> /ROW1
- D15 pad 1: /left/ROW2 -> /ROW2
- D16 pad 1: /left/ROW3 -> /ROW3
- D17 pad 1: /left/ROW0 -> /ROW0
- D18 pad 1: /left/ROW1 -> /ROW1
- D19 pad 1: /left/ROW2 -> /ROW2
- D2 pad 1: /left/ROW1 -> /ROW1
- D20 pad 1: /left/ROW3 -> /ROW3
- D21 pad 1: /right/ROW0 -> /ROW0
- D22 pad 1: /right/ROW1 -> /ROW1
- D23 pad 1: /right/ROW2 -> /ROW2
- D24 pad 1: /right/ROW0 -> /ROW0
- D25 pad 1: /right/ROW1 -> /ROW1
- D26 pad 1: /right/ROW2 -> /ROW2
- D27 pad 1: /right/ROW0 -> /ROW0
- D28 pad 1: /right/ROW1 -> /ROW1
- D29 pad 1: /right/ROW2 -> /ROW2
- D3 pad 1: /left/ROW2 -> /ROW2
- D30 pad 1: /right/ROW0 -> /ROW0
- D31 pad 1: /right/ROW1 -> /ROW1
- D32 pad 1: /right/ROW2 -> /ROW2
- D33 pad 1: /right/ROW0 -> /ROW0
- D34 pad 1: /right/ROW1 -> /ROW1
- D35 pad 1: /right/ROW2 -> /ROW2
- D36 pad 1: /right/ROW3 -> /ROW3
- D37 pad 1: /right/ROW0 -> /ROW0
- D38 pad 1: /right/ROW1 -> /ROW1
- D39 pad 1: /right/ROW2 -> /ROW2
- D4 pad 1: /left/ROW0 -> /ROW0
- D40 pad 1: /right/ROW3 -> /ROW3
- D5 pad 1: /left/ROW1 -> /ROW1
- D6 pad 1: /left/ROW2 -> /ROW2
- D7 pad 1: /left/ROW0 -> /ROW0
- D8 pad 1: /left/ROW1 -> /ROW1
- D9 pad 1: /left/ROW2 -> /ROW2
- SW1 pad 1: /left/COL0 -> /COL0
- SW10 pad 1: /left/COL3 -> /COL3
- SW11 pad 1: /left/COL3 -> /COL3
- SW12 pad 1: /left/COL3 -> /COL3
- SW13 pad 1: /left/COL4 -> /COL4
- SW14 pad 1: /left/COL4 -> /COL4
- SW15 pad 1: /left/COL4 -> /COL4
- SW16 pad 1: /left/COL4 -> /COL4
- SW17 pad 1: /left/COL5 -> /COL5
- SW18 pad 1: /left/COL5 -> /COL5
- SW19 pad 1: /left/COL5 -> /COL5
- SW2 pad 1: /left/COL0 -> /COL0
- SW20 pad 1: /left/COL5 -> /COL5
- SW21 pad 1: /right/COL0 -> /COL0
- SW22 pad 1: /right/COL0 -> /COL0
- SW23 pad 1: /right/COL0 -> /COL0
- SW24 pad 1: /right/COL1 -> /COL1
- SW25 pad 1: /right/COL1 -> /COL1
- SW26 pad 1: /right/COL1 -> /COL1
- SW27 pad 1: /right/COL2 -> /COL2
- SW28 pad 1: /right/COL2 -> /COL2
- SW29 pad 1: /right/COL2 -> /COL2
- SW3 pad 1: /left/COL0 -> /COL0
- SW30 pad 1: /right/COL3 -> /COL3
- SW31 pad 1: /right/COL3 -> /COL3
- SW32 pad 1: /right/COL3 -> /COL3
- SW33 pad 1: /right/COL4 -> /COL4
- SW34 pad 1: /right/COL4 -> /COL4
- SW35 pad 1: /right/COL4 -> /COL4
- SW36 pad 1: /right/COL4 -> /COL4
- SW37 pad 1: /right/COL5 -> /COL5
- SW38 pad 1: /right/COL5 -> /COL5
- SW39 pad 1: /right/COL5 -> /COL5
- SW4 pad 1: /left/COL1 -> /COL1
- SW40 pad 1: /right/COL5 -> /COL5
- SW5 pad 1: /left/COL1 -> /COL1
- SW6 pad 1: /left/COL1 -> /COL1
- SW7 pad 1: /left/COL2 -> /COL2
- SW8 pad 1: /left/COL2 -> /COL2
- SW9 pad 1: /left/COL2 -> /COL2
- U1 pad 10: /left/ROW1 -> /ROW1
- U1 pad 11: /left/ROW0 -> /ROW0
- U1 pad 2: /left/COL0 -> /COL0
- U1 pad 3: /left/COL1 -> /COL1
- U1 pad 4: /left/COL2 -> /COL2
- U1 pad 5: /left/COL3 -> /COL3
- U1 pad 6: /left/COL4 -> /COL4
- U1 pad 7: /left/COL5 -> /COL5
- U1 pad 8: /left/ROW3 -> /ROW3
- U1 pad 9: /left/ROW2 -> /ROW2
- U2 pad 10: /right/ROW1 -> /ROW1
- U2 pad 11: /right/ROW0 -> /ROW0
- U2 pad 2: /right/COL0 -> /COL0
- U2 pad 3: /right/COL1 -> /COL1
- U2 pad 4: /right/COL2 -> /COL2
- U2 pad 5: /right/COL3 -> /COL3
- U2 pad 6: /right/COL4 -> /COL4
- U2 pad 7: /right/COL5 -> /COL5
- U2 pad 8: /right/ROW3 -> /ROW3
- U2 pad 9: /right/ROW2 -> /ROW2
Routing:
- net /COL5: track 0.00 -> 324.5 mm
- net /COL4: track 0.00 -> 313.8 mm
- net /ROW2: track 0.00 -> 276.3 mm
- net /ROW0: track 0.00 -> 268.7 mm
- net /COL2: track 0.00 -> 263.9 mm
- net /COL1: track 0.00 -> 261.9 mm
- net /COL0: track 0.00 -> 261.2 mm
- net /COL3: track 0.00 -> 259.6 mm
- net /ROW1: track 0.00 -> 255.3 mm
- net /right/COL5: track 194.5 -> 0.00 mm
- net /left/COL0: track 188.4 -> 0.00 mm
- net /left/COL1: track 168.0 -> 0.00 mm
- net /right/COL4: track 163.3 -> 0.00 mm
- net /left/COL4: track 150.5 -> 0.00 mm
- net /left/COL2: track 149.0 -> 0.00 mm
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
Commit message: feat: new journal, fix some errors, usb-c interconnect, new edge cuts and so much more
Parts:
- B1, B2, B3, B4, B5: footprint PCM_marbastlib-various:mousebites_2mm -> kicad_care_package:mousebites_2mm
- moved D51 115.7 mm to (159.5, 145.0)
- moved SW51 115.7 mm to (159.4, 135.5)
- moved D50 115.7 mm to (138.0, 142.1)
- moved SW50 115.7 mm to (137.5, 132.6)
- moved D40 18.5 mm to (178.5, 144.0)
- moved SW40 18.5 mm to (178.5, 134.6)
- moved D20 18.5 mm to (118.5, 144.6)
- moved SW20 18.5 mm to (118.5, 135.1)
- moved H2 18.5 mm to (82.5, 127.5)
- moved SW16 17.6 mm to (99.5, 131.5)
- moved D36 17.5 mm to (197.5, 142.0)
- moved SW36 17.5 mm to (197.5, 132.6)
- moved D16 17.2 mm to (100.0, 141.0)
- moved H5 14.1 mm to (211.0, 131.5)
- moved H1 12.1 mm to (130.0, 113.5)
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Routing:
- net Net-(D16-A): track 4.84 -> 0.00 mm
- net Net-(D50-A): track 0.00 -> 4.80 mm
- net Net-(D51-A): track 0.00 -> 4.70 mm
- net Net-(D36-A): track 4.70 -> 0.00 mm
Other:
- board size 273 x 89.5 mm -> 273 x 105.5 mm

Commit message: feat: interconnect cable, new journal
Routing:
- net /COL0: track 261.2 -> 455.7 mm
- net /COL5: track 324.5 -> 130.1 mm

Commit message: feat: new journal, finish PCB
Parts:
- removed B5: MouseBite, kicad_care_package:mousebites_2mm
- added G***: LOGO, LOGO, F.Cu at (230.5, 125.3)
- added P1: USB_C_Plug_USB2.0, Connector_USB:USB_C_Receptacle_GCT_USB4105-xx-A_16P_TopMnt_Horizontal, F.Cu at (143.8, 115.5)
- added P2: USB_C_Plug_USB2.0, Connector_USB:USB_C_Receptacle_GCT_USB4105-xx-A_16P_TopMnt_Horizontal, F.Cu at (153.2, 115.5)
- added R1: 4.7k, Resistor_SMD:R_0805_2012Metric_Pad1.20x1.40mm_HandSolder, F.Cu at (142.5, 122.0)
- moved B3 27.1 mm to (149.4, 144.4), turned to 0 degrees
- moved B1 13.6 mm to (149.4, 90.5), turned to 0 degrees
- moved B2 13.5 mm to (149.4, 103.8), turned to 0 degrees
- moved H4 7.21 mm to (163.0, 117.5)
- moved SW51 5.00 mm to (159.5, 130.5)
- moved D51 5.00 mm to (159.5, 140.0)
- moved H5 4.03 mm to (211.5, 127.5)
- moved H2 3.00 mm to (85.5, 127.5)
- moved D50 2.16 mm to (137.5, 140.0)
- moved SW50 2.10 mm to (137.5, 130.5)
- moved B4 1.96 mm to (149.4, 131.4), turned to 0 degrees
- moved SW1 1.50 mm to (22.0, 81.5)
- moved SW2 1.00 mm to (22.0, 100.5)
- moved D16 1.00 mm to (100.0, 142.0)
- moved D40 1.00 mm to (178.5, 145.0)
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Connections:
- D21 pad 1: /ROW0 -> /ROW4
- D22 pad 1: /ROW1 -> /ROW5
- D23 pad 1: /ROW2 -> /ROW6
- D24 pad 1: /ROW0 -> /ROW4
- D25 pad 1: /ROW1 -> /ROW5
- D26 pad 1: /ROW2 -> /ROW6
- D27 pad 1: /ROW0 -> /ROW4
- D28 pad 1: /ROW1 -> /ROW5
- D29 pad 1: /ROW2 -> /ROW6
- D30 pad 1: /ROW0 -> /ROW4
- D31 pad 1: /ROW1 -> /ROW5
- D32 pad 1: /ROW2 -> /ROW6
- D33 pad 1: /ROW0 -> /ROW4
- D34 pad 1: /ROW1 -> /ROW5
- D35 pad 1: /ROW2 -> /ROW6
- D36 pad 1: /ROW3 -> /ROW7
- D37 pad 1: /ROW0 -> /ROW4
- D38 pad 1: /ROW1 -> /ROW5
- D39 pad 1: /ROW2 -> /ROW6
- D40 pad 1: /ROW3 -> /ROW7
- D51 pad 1: /ROW3 -> /ROW7
- SW16 pad 1: /COL4 -> /COL3
- SW20 pad 1: /COL5 -> /COL4
- SW21 pad 1: /COL0 -> /COL6
- SW22 pad 1: /COL0 -> /COL6
- SW23 pad 1: /COL0 -> /COL6
- SW24 pad 1: /COL1 -> /COL7
- SW25 pad 1: /COL1 -> /COL7
- SW26 pad 1: /COL1 -> /COL7
- SW27 pad 1: /COL2 -> /COL8
- SW28 pad 1: /COL2 -> /COL8
- SW29 pad 1: /COL2 -> /COL8
- SW30 pad 1: /COL3 -> /COL9
- SW31 pad 1: /COL3 -> /COL9
- SW32 pad 1: /COL3 -> /COL9
- SW33 pad 1: /COL4 -> /COL10
- SW34 pad 1: /COL4 -> /COL10
- SW35 pad 1: /COL4 -> /COL10
- SW36 pad 1: /COL4 -> /COL9
- SW37 pad 1: /COL5 -> /COL11
- SW38 pad 1: /COL5 -> /COL11
- SW39 pad 1: /COL5 -> /COL11
- SW40 pad 1: /COL5 -> /COL10
- SW50 pad 1: /COL0 -> /COL5
- SW51 pad 1: /COL0 -> /COL11
- U1 pad 1: unconnected-(U1-GPIO26/ADC0/A0-Pad1)_1 -> /INTERCON_L
- U1 pad 10: /ROW1 -> /COL3
- U1 pad 11: /ROW0 -> /COL2
- U1 pad 12: unconnected-(U1-3V3-Pad12)_1 -> /3V3_L
- U1 pad 13: unconnected-(U1-GND-Pad13) -> /GND_L
- U1 pad 14: unconnected-(U1-VBUS-Pad14) -> /5V_L
- U1 pad 2: /COL0 -> /ROW0
- U1 pad 3: /COL1 -> /ROW1
- U1 pad 4: /COL2 -> /ROW2
- U1 pad 5: /COL3 -> /ROW3
- U1 pad 6: /COL4 -> /COL0
- U1 pad 7: /COL5 -> /COL1
- U1 pad 8: /ROW3 -> /COL5
- U1 pad 9: /ROW2 -> /COL4
- U2 pad 1: unconnected-(U2-GPIO26/ADC0/A0-Pad1) -> /INTERCON_R
- U2 pad 10: /ROW1 -> /ROW5
- U2 pad 11: /ROW0 -> /ROW4
- U2 pad 13: unconnected-(U2-GND-Pad13) -> /GND_R
- U2 pad 14: unconnected-(U2-VBUS-Pad14) -> /5V_R
- U2 pad 2: /COL0 -> /COL6
- U2 pad 3: /COL1 -> /COL7
- U2 pad 4: /COL2 -> /COL8
- U2 pad 5: /COL3 -> /COL9
- U2 pad 6: /COL4 -> /COL10
- U2 pad 7: /COL5 -> /COL11
- U2 pad 8: /ROW3 -> /ROW7
- U2 pad 9: /ROW2 -> /ROW6
Routing:
- net /COL0: track 455.7 -> 199.2 mm
- net /COL11: track 0.00 -> 196.5 mm
- net /COL10: track 0.00 -> 170.0 mm
- net /COL4: track 313.8 -> 168.3 mm
- net /ROW0: track 268.7 -> 124.3 mm
- net /COL9: track 0.00 -> 140.9 mm
- net /ROW2: track 276.3 -> 136.0 mm
- net /ROW1: track 255.3 -> 126.7 mm
- net /ROW6: track 0.00 -> 126.9 mm
- net /ROW4: track 0.00 -> 123.5 mm
- net /COL8: track 0.00 -> 120.2 mm
- net /ROW5: track 0.00 -> 114.1 mm
- net /COL7: track 0.00 -> 100.0 mm
- net /COL2: track 263.9 -> 178.4 mm
- net /COL1: track 261.9 -> 179.3 mm
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- added copper zone on B.Cu, net /GND_L
- added copper zone on B.Cu, net /GND_R
Other:
- board size 273 x 105.5 mm -> 273 x 89.5 mm

Commit message: feat: switch to 5.1k resistor, fix all 3D models
Parts:
- moved H1 4.19 mm to (130.5, 117.5)
- moved H4 0.50 mm to (162.5, 117.5)
Routing:
- net /ROW1: track 126.7 -> 125.3 mm

Commit message: chore: impove traces, cleanup
Parts:
- moved G*** 0.55 mm to (230.5, 125.8)
- moved D50 0.50 mm to (137.5, 139.5)
- moved D51 0.50 mm to (159.5, 139.5)
- moved SW50 0.50 mm to (137.5, 130.0)
- moved SW51 0.30 mm to (159.5, 130.2)
Routing:
- net /COL11: track 196.5 -> 195.5 mm
- net /ROW0: track 124.3 -> 123.3 mm

Commit message: feat: gerbers, new journal, update readme, finish BOM
Parts:
- removed H5, H6: MountingHole, MountingHole:MountingHole_2.2mm_M2
- R1: value 4.7k -> 5.1k
- moved H4 100.8 mm to (250.0, 67.5)
- moved H1 81.6 mm to (211.5, 127.5)
