File: NordBoard.kicad_pcb (KiCad board)
At the start: 2 copper layers, 273 x 89.5 mm, 98 parts, among them P1 USB_C_Plug_USB2.0, P2 USB_C_Plug_USB2.0, SW1 SW_Push, SW10 SW_Push, SW11 SW_Push, SW12 SW_Push, SW13 SW_Push, SW14 SW_Push, SW15 SW_Push, SW16 SW_Push, SW17 SW_Push, SW18 SW_Push, SW19 SW_Push, SW2 SW_Push, SW20 SW_Push, SW21 SW_Push, SW22 SW_Push, SW23 SW_Push, SW24 SW_Push, SW25 SW_Push, SW26 SW_Push, SW27 SW_Push, SW28 SW_Push, SW29 SW_Push, SW3 SW_Push, SW30 SW_Push, SW31 SW_Push, SW32 SW_Push, SW33 SW_Push, SW34 SW_Push, SW35 SW_Push, SW36 SW_Push, SW37 SW_Push, SW38 SW_Push, SW39 SW_Push, SW4 SW_Push, SW40 SW_Push, SW5 SW_Push, SW50 SW_Push, SW51 SW_Push, SW6 SW_Push, SW7 SW_Push, SW8 SW_Push, SW9 SW_Push, U1 XIAO-RP2040-DIP, U2 XIAO-RP2040-DIP

Commit message: feat: switch away from mousebites to reduce cost
Parts:
- removed B1, B2, B3, B4: MouseBite, kicad_care_package:mousebites_2mm
- moved P1 3.32 mm to (140.5, 115.5)
- moved D37 1.84 mm to (273.2, 90.9)
- moved D38 1.84 mm to (273.3, 110.0)
- moved SW37 1.84 mm to (273.3, 81.6)
- moved SW38 1.84 mm to (273.3, 100.7)
- moved SW39 1.84 mm to (273.3, 119.8)
- moved D21 1.84 mm to (178.2, 84.9)
- moved D22 1.84 mm to (178.2, 103.9)
- moved D23 1.84 mm to (178.1, 122.9)
- moved D24 1.84 mm to (197.2, 80.7)
- moved D25 1.84 mm to (197.2, 99.7)
- moved D26 1.84 mm to (197.2, 118.7)
- moved D27 1.84 mm to (216.2, 77.3)
- moved D28 1.84 mm to (216.2, 96.3)
- moved D29 1.84 mm to (216.2, 115.3)
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Routing:
- net /GND_R: track 58.4 -> 11.6 mm
- net /GND_L: track 36.8 -> 12.4 mm
- net /INTERCON_L: track 47.3 -> 54.3 mm
- net /INTERCON_R: track 28.9 -> 35.6 mm
- net /5V_L: track 29.9 -> 31.4 mm
- net /COL10: track 170.0 -> 169.0 mm
- net /5V_R: track 32.7 -> 31.8 mm
- net /COL5: track 141.1 -> 140.2 mm
- net /COL4: track 168.3 -> 167.4 mm
- net /COL2: track 178.4 -> 179.1 mm
- net /COL11: track 195.5 -> 194.8 mm
Other:
- board size 273 x 89.5 mm -> 271.2 x 89.5 mm
