File: NordBoard.kicad_pcb (KiCad board)
At the start: 2 copper layers, 271.2 x 89.5 mm, 94 parts, among them P1 USB_C_Plug_USB2.0, P2 USB_C_Plug_USB2.0, SW1 SW_Push, SW10 SW_Push, SW11 SW_Push, SW12 SW_Push, SW13 SW_Push, SW14 SW_Push, SW15 SW_Push, SW16 SW_Push, SW17 SW_Push, SW18 SW_Push, SW19 SW_Push, SW2 SW_Push, SW20 SW_Push, SW21 SW_Push, SW22 SW_Push, SW23 SW_Push, SW24 SW_Push, SW25 SW_Push, SW26 SW_Push, SW27 SW_Push, SW28 SW_Push, SW29 SW_Push, SW3 SW_Push, SW30 SW_Push, SW31 SW_Push, SW32 SW_Push, SW33 SW_Push, SW34 SW_Push, SW35 SW_Push, SW36 SW_Push, SW37 SW_Push, SW38 SW_Push, SW39 SW_Push, SW4 SW_Push, SW40 SW_Push, SW5 SW_Push, SW50 SW_Push, SW51 SW_Push, SW6 SW_Push, SW7 SW_Push, SW8 SW_Push, SW9 SW_Push, U1 XIAO-RP2040-DIP, U2 XIAO-RP2040-DIP

Commit message: feat: finish schematic, new journal entry
Parts:
- removed U2: XIAO-RP2040-DIP, kicad_care_package:XIAO-RP2040-DIP
- added C2: 100nF, Capacitor_SMD:C_0603_1608Metric, F.Cu at (156.2, 80.8)
- added C5: 4.7uF, Capacitor_SMD:C_0805_2012Metric, F.Cu at (151.7, 91.5)
- added P3: USB_C_Plug_USB2.0, Connector_USB:USB_C_Receptacle_HRO_TYPE-C-31-M-12, F.Cu at (148.4, 85.3)
- added R2: 5.1kO, Resistor_SMD:R_0603_1608Metric, F.Cu at (156.2, 85.8)
- added R3: 1k, Resistor_SMD:R_0603_1608Metric, F.Cu at (156.2, 88.3)
- added S1: SKRPACE010, SKRPACE010:SW_SKRPACE010, F.Cu at (146.1, 92.3)
- added TP1: TestPoint, TestPoint:TestPoint_Pad_D1.0mm, F.Cu at (141.0, 81.0)
- added TP2: TestPoint, TestPoint:TestPoint_Pad_D1.0mm, F.Cu at (141.0, 84.1)
- added TP3: TestPoint, TestPoint:TestPoint_Pad_D1.0mm, F.Cu at (141.0, 87.1)
- added TP4: TestPoint, TestPoint:TestPoint_Pad_D1.0mm, F.Cu at (141.0, 90.2)
- P1, P2: footprint Connector_USB:USB_C_Receptacle_GCT_USB4105-xx-A_16P_TopMnt_Horizontal -> Connector_USB:USB_C_Receptacle_Molex_105450-0101
- R1: value 5.1k -> 5.1kO; footprint Resistor_SMD:R_0805_2012Metric_Pad1.20x1.40mm_HandSolder -> Resistor_SMD:R_0603_1608Metric
- U1: value XIAO-RP2040-DIP -> CH32X035DS0; footprint kicad_care_package:XIAO-RP2040-DIP -> Package_DFN_QFN:WQFN-28-1EP_4x4mm_P0.4mm_EP2.7x2.7mm
- moved R1 41.1 mm to (156.2, 83.3)
Connections:
- P1 pad A1: /GND_L -> GND
- P1 pad A12: /GND_L -> GND
- P1 pad A4: /5V_L -> unconnected-(P1-VBUS-PadA4)_1
- P1 pad A6: /INTERCON_L -> /COL0
- P1 pad A7: unconnected-(P1-D--PadA7) -> /COL1
- P1 pad A9: /5V_L -> unconnected-(P1-VBUS-PadA4)
- P1 pad B1: /GND_L -> GND
- P1 pad B12: /GND_L -> GND
- P1 pad B4: /5V_L -> unconnected-(P1-VBUS-PadA4)_2
- P1 pad B6: /INTERCON_L -> /COL0
- P1 pad B7: unconnected-(P1-D--PadB7) -> /COL1
- P1 pad B9: /5V_L -> unconnected-(P1-VBUS-PadA4)_3
- P1 pad SH: /GND_L -> GND
- P2 pad A1: /GND_R -> GND
- P2 pad A12: /GND_R -> GND
- P2 pad A4: /5V_R -> unconnected-(P2-VBUS-PadA4)_1
- P2 pad A6: /INTERCON_R -> /COL0
- P2 pad A7: unconnected-(P2-D--PadA7) -> /COL1
- P2 pad A9: /5V_R -> unconnected-(P2-VBUS-PadA4)_3
- P2 pad B1: /GND_R -> GND
- P2 pad B12: /GND_R -> GND
- P2 pad B4: /5V_R -> unconnected-(P2-VBUS-PadA4)_2
- P2 pad B6: /INTERCON_R -> /COL0
- P2 pad B7: unconnected-(P2-D--PadB7) -> /COL1
- P2 pad B9: /5V_R -> unconnected-(P2-VBUS-PadA4)
- P2 pad SH: /GND_R -> GND
- R1 pad 1: /INTERCON_L -> Net-(P3-CC1)
- R1 pad 2: /3V3_L -> GND
- SW21 pad 1: /COL6 -> /COL0
- SW22 pad 1: /COL6 -> /COL0
- SW23 pad 1: /COL6 -> /COL0
- SW24 pad 1: /COL7 -> /COL1
- SW25 pad 1: /COL7 -> /COL1
- SW26 pad 1: /COL7 -> /COL1
- SW27 pad 1: /COL8 -> /COL2
- SW28 pad 1: /COL8 -> /COL2
- SW29 pad 1: /COL8 -> /COL2
- SW30 pad 1: /COL9 -> /COL3
- SW31 pad 1: /COL9 -> /COL3
- SW32 pad 1: /COL9 -> /COL3
- SW33 pad 1: /COL10 -> /COL4
- SW34 pad 1: /COL10 -> /COL4
- SW35 pad 1: /COL10 -> /COL4
- SW36 pad 1: /COL9 -> /COL3
- SW37 pad 1: /COL11 -> /COL5
- SW38 pad 1: /COL11 -> /COL5
- SW39 pad 1: /COL11 -> /COL5
- SW40 pad 1: /COL10 -> /COL4
- SW51 pad 1: /COL11 -> /COL5
- U1 pad 1: /INTERCON_L -> unconnected-(U1-PC15/CC2-Pad1)
- U1 pad 10: /COL3 -> /COL5
- U1 pad 11: /COL2 -> unconnected-(U1-PA6-Pad11)
- U1 pad 12: /3V3_L -> unconnected-(U1-PA7-Pad12)
- U1 pad 13: /GND_L -> /ROW0
- U1 pad 14: /5V_L -> /ROW1
- U1 pad 2: /ROW0 -> +5V
- U1 pad 3: /ROW1 -> unconnected-(U1-PC0-Pad3)
- U1 pad 4: /ROW2 -> unconnected-(U1-PC3-Pad4)
- U1 pad 5: /ROW3 -> /COL0
- U1 pad 6: /COL0 -> /COL1
- U1 pad 7: /COL1 -> /COL2
- U1 pad 8: /COL5 -> /COL3
Routing:
- net /COL5: track 140.2 -> 341.6 mm
- net /COL11: track 201.4 -> 0.00 mm
- net /COL4: track 167.4 -> 337.3 mm
- net /COL10: track 169.9 -> 0.00 mm
- net /COL3: track 190.6 -> 330.8 mm
- net /COL9: track 140.2 -> 0.00 mm
- net /COL8: track 113.9 -> 0.00 mm
- net /COL2: track 179.1 -> 293.0 mm
- net /COL7: track 95.3 -> 0.00 mm
- net /COL1: track 179.3 -> 274.6 mm
- net /COL0: track 199.2 -> 272.7 mm
- net /COL6: track 73.4 -> 0.00 mm
- net GND: track 0.00 -> 28.8 mm, vias 0 -> 1
- net /GND_R: track 22.8 -> 0.00 mm, vias 1 -> 0
- net /GND_L: track 23.3 -> 17.2 mm
- added copper zone on B.Cu, net GND
- added copper zone on B.Cu, net unconnected-(U1-PB1/PB5-Pad16)
- removed copper zone on B.Cu, net /GND_L
- removed copper zone on B.Cu, net /GND_R

Commit message: e
Parts:
- moved R3 107.6 mm to (55.5, 126.0)
- moved R1 93.1 mm to (72.3, 123.5)
- moved C2 79.8 mm to (86.7, 120.0)
- moved TP1 77.4 mm to (68.5, 108.0), turned to 90 degrees
- moved TP2 77.4 mm to (68.5, 111.0), turned to 90 degrees
- moved TP3 77.3 mm to (68.5, 114.0), turned to 90 degrees
- moved C5 75.4 mm to (83.5, 123.5)
- moved R2 75.1 mm to (90.5, 122.0)
- moved TP4 74.0 mm to (68.5, 105.0), turned to 90 degrees
- moved S1 72.8 mm to (79.0, 120.5)
- moved 1 63.3 mm to (78.7, 127.5)
- moved P3 23.4 mm to (134.3, 104.0), turned to 180 degrees
- moved H2 8.56 mm to (86.5, 136.0)
- renumbered U1 to 1
Routing:
- net /ROW0: track 123.3 -> 230.1 mm
- net /ROW6: track 126.9 -> 189.2 mm
- net /INTERCON_L: track 54.3 -> 0.00 mm
- net /COL3: track 330.8 -> 276.8 mm, vias 0 -> 1
- net /COL4: track 337.3 -> 286.3 mm
- net /COL5: track 341.6 -> 297.7 mm
- net /INTERCON_R: track 36.6 -> 0.00 mm
- net /COL2: track 293.0 -> 257.7 mm, vias 0 -> 1
- net /5V_R: track 31.6 -> 0.00 mm
- net /5V_L: track 31.4 -> 0.00 mm
- net /ROW7: track 78.9 -> 105.0 mm
- net /3V3_L: track 25.9 -> 0.00 mm
- net /ROW1: track 125.3 -> 147.5 mm, vias 0 -> 2
- net /COL1: track 274.6 -> 256.2 mm, vias 0 -> 1
- net /ROW3: track 82.6 -> 64.8 mm
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Other:
- board text added: "5V"
- board text added: "GND"
- board text added: "RX"
- board text added: "TX"
- board text added: "snowdrift"
- board text removed: "NordBoard"

Commit message: feat: new journal, more routing
Parts:
- moved R1 63.8 mm to (135.0, 111.5), turned to -90 degrees
- moved R2 43.8 mm to (133.0, 111.5), turned to -90 degrees
- moved H2 35.4 mm to (52.0, 128.0)
- moved R3 20.3 mm to (75.0, 120.5), turned to 90 degrees
- moved C2 13.0 mm to (75.0, 125.5), turned to 90 degrees
- moved C5 10.7 mm to (73.0, 125.5), turned to 90 degrees
Routing:
- net /COL5: track 297.7 -> 383.3 mm, vias 0 -> 7
- net +5V: track 0.00 -> 84.6 mm, vias 0 -> 2
- net /COL4: track 286.3 -> 366.8 mm, vias 0 -> 3
- net /COL0: track 258.1 -> 338.4 mm, vias 1 -> 3
- net /ROW4: track 129.3 -> 208.8 mm, vias 0 -> 2
- net /ROW5: track 121.0 -> 195.8 mm, vias 0 -> 2
- net /DATA0: track 0.00 -> 71.7 mm, vias 0 -> 2
- net /COL1: track 256.2 -> 320.9 mm, vias 1 -> 6
- net /COL3: track 276.8 -> 336.8 mm, vias 1 -> 3
- net /COL2: track 257.7 -> 304.1 mm, vias 1 -> 3
- net /DATA1: track 0.00 -> 30.0 mm
- net /ROW7: track 105.0 -> 133.1 mm, vias 0 -> 2
- net GND: track 36.4 -> 10.6 mm, vias 0 -> 5
- net Net-(U1-PC18/DIO): track 0.00 -> 19.4 mm, vias 0 -> 2
- net /ROW6: track 189.2 -> 205.1 mm, vias 0 -> 4
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Other:
- outline, holes or cut-outs redrawn

Commit message: feat: alomst finish new PCB routing
Parts:
- removed S1: SKRPACE010, SKRPACE010:SW_SKRPACE010
- added SW41: SW_Push, Jumper:SolderJumper-2_P1.3mm_Open_Pad1.0x1.5mm, F.Cu at (125.2, 89.9)
- moved C5 58.8 mm to (125.0, 98.0)
- moved R3 56.4 mm to (125.0, 94.5)
- moved U1 56.1 mm to (130.2, 105.2)
- moved C2 54.7 mm to (125.0, 103.2)
- moved H2 31.0 mm to (83.0, 128.0)
- moved R1 9.38 mm to (134.0, 102.2)
- moved P3 6.31 mm to (140.6, 103.9)
- moved R2 3.95 mm to (134.0, 107.7)
- renumbered 1 to U1
Connections:
- R3 pad 2: GND -> Net-(SW41-A)
Routing:
- net /COL5: track 383.3 -> 301.2 mm
- net /ROW0: track 229.8 -> 151.4 mm, vias 0 -> 2
- net Net-(U1-PC19/DCK): track 0.00 -> 78.0 mm, vias 0 -> 2
- net /COL0: track 338.4 -> 278.3 mm
- net /ROW6: track 205.1 -> 148.8 mm
- net Net-(U1-PC18/DIO): track 19.4 -> 69.3 mm
- net /ROW7: track 133.1 -> 84.4 mm, vias 2 -> 4
- net /DATA0: track 71.7 -> 23.6 mm, vias 2 -> 0
- net /ROW5: track 195.8 -> 151.4 mm
- net /ROW4: track 208.8 -> 168.1 mm
- net /COL1: track 320.9 -> 282.3 mm
- net /COL4: track 366.8 -> 334.4 mm
- net +5V: track 84.6 -> 116.2 mm, vias 2 -> 0
- net /COL2: track 304.1 -> 281.4 mm, vias 3 -> 4
- net /ROW3: track 64.8 -> 81.4 mm
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- added copper zone on F.Cu, net GND
- removed copper zone on B.Cu, net unconnected-(U1-PB1/PB5-Pad16)
Other:
- board size 271.2 x 89.5 mm -> 270.5 x 89 mm
- board text added: "snowlayer"
- board text removed: "snowdrift"

Commit message: feat: new journal, rename project, finish PCB
Parts:
- moved P3 1.12 mm to (140.1, 104.9)
- moved R1 1.12 mm to (133.5, 103.2)
- moved R2 1.12 mm to (133.5, 108.7)
- moved U1 1.12 mm to (129.7, 106.2)
- moved C2 1.04 mm to (126.0, 103.5)
Routing:
- net GND: track 25.4 -> 31.9 mm, vias 5 -> 21
- net /ROW2: track 140.1 -> 134.3 mm
- net +5V: track 116.2 -> 112.1 mm
- net /DATA1: track 36.9 -> 39.6 mm
- net Net-(U1-PC18/DIO): track 69.3 -> 66.6 mm
- net /COL4: track 334.4 -> 332.0 mm
- net /COL3: track 323.5 -> 321.8 mm
- net /ROW1: track 134.3 -> 132.7 mm
- net /ROW3: track 81.4 -> 80.0 mm
- net /ROW0: track 151.4 -> 150.2 mm
- net Net-(P3-CC1): track 12.2 -> 13.3 mm
- net /ROW7: track 84.4 -> 83.3 mm
- net /ROW4: track 168.1 -> 167.2 mm
- net /ROW5: track 151.4 -> 150.5 mm
- net /COL0: track 278.3 -> 277.5 mm
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Other:
- outline, holes or cut-outs redrawn
- board text added: "P2"
