File: NordBoard.kicad_sch (KiCad schematic)
At the start: 97 parts, among them P1 USB_C_Plug_USB2.0, P2 USB_C_Plug_USB2.0, SW1 SW_Push, SW10 SW_Push, SW11 SW_Push, SW12 SW_Push, SW13 SW_Push, SW14 SW_Push, SW15 SW_Push, SW16 SW_Push, SW17 SW_Push, SW18 SW_Push, SW19 SW_Push, SW2 SW_Push, SW20 SW_Push, SW21 SW_Push, SW22 SW_Push, SW23 SW_Push, SW24 SW_Push, SW25 SW_Push, SW26 SW_Push, SW27 SW_Push, SW28 SW_Push, SW29 SW_Push, SW3 SW_Push, SW30 SW_Push, SW31 SW_Push, SW32 SW_Push, SW33 SW_Push, SW34 SW_Push, SW35 SW_Push, SW36 SW_Push, SW37 SW_Push, SW38 SW_Push, SW39 SW_Push, SW4 SW_Push, SW40 SW_Push, SW5 SW_Push, SW50 SW_Push, SW51 SW_Push, SW6 SW_Push, SW7 SW_Push, SW8 SW_Push, SW9 SW_Push, U1 XIAO-RP2040-DIP, U2 XIAO-RP2040-DIP

Commit message: feat: switch away from mousebites to reduce cost
Parts:
- removed B1, B2, B3, B4: MouseBite, kicad_care_package:mousebites_2mm, symbol Mechanical:MouseBite
Other:
- note added: "Left Interconnect"
- note added: "Right Interconnect"
- note removed: "Mousebites"
- note removed: "USB-C Interconnect"

Commit message: feat: new journal, switch to new interconnect and MCU
Parts:
- removed R1: 5.1k, Resistor_SMD:R_0805_2012Metric_Pad1.20x1.40mm_HandSolder, symbol Device:R
- removed U2: XIAO-RP2040-DIP, kicad_care_package:XIAO-RP2040-DIP, symbol XIAO_RP2040:MOUDLE-SEEEDUINO-XIAO
- P1, P2: footprint Connector_USB:USB_C_Receptacle_GCT_USB4105-xx-A_16P_TopMnt_Horizontal -> Connector_USB:USB_C_Receptacle_GCT_USB4105; symbol Connector:USB_C_Receptacle_USB2.0_16P -> Connector:USB_C_Receptacle
- U1: footprint kicad_care_package:XIAO-RP2040-DIP -> Package_QFP:LQFP-32_7x7mm_P0.8mm; symbol XIAO_RP2040:MOUDLE-SEEEDUINO-XIAO -> MCU_ST_STM32F0:STM32F042K6Tx
Connections:
- net 3V3_L: no longer U1.12 (3V3)
- net 5V_L: no longer P1.A4 (VBUS), P1.A9 (VBUS), P1.B4 (VBUS), P1.B9 (VBUS), U1.14 (5V)
- net COL2: now also U1.8 (PA2); no longer U1.11 (PA6_A10_D10_MOSI)
- net COL3: now also U1.9 (PA3); no longer U1.10 (PA5_A9_D9_MISO)
- net COL4: now also U1.10 (PA4); no longer U1.9 (PA7_A8_D8_SCK)
- net COL5: now also U1.11 (PA5); no longer U1.8 (PB09_A7_D7_RX)
- net GND_L: no longer U1.13 (GND)
- net ROW0: now also U1.14 (PB0); no longer U1.2 (PA4_A1_D1)
- net ROW1: now also U1.15 (PB1); no longer U1.3 (PA10_A2_D2)
- net ROW2: now also U1.26 (PB3); no longer U1.4 (PA11_A3_D3)
- net ROW3: now also U1.27 (PB4); no longer U1.5 (PA8_A4_D4_SDA)
- net ROW4: now also U1.28 (PB5)
- net ROW5: now also U1.29 (PB6)
- net ROW6: now also U1.30 (PB7)
- net ROW7: now also U1.31 (PB8)
- net 5V_R: no longer names the net of P2.A4 (VBUS), P2.A9 (VBUS), P2.B4 (VBUS), P2.B9 (VBUS)
- removed net INTERCON_L: P1.A6 (D+), P1.B6 (D+), U1.1 (PA02_A0_D0)
- net INTERCON_R: no longer names the net of P2.A6 (D+)
- net INTERCON_R: no longer P2.B6 (D+)
- new net: P1.A4 (VBUS), P1.A9 (VBUS), P1.B4 (VBUS), P1.B9 (VBUS)
- no-connect marks 13 -> 0
Other:
- note added: "Left MCU"
- note removed: "Interconnect Resistor"
- note removed: "Left Xiao"
- note removed: "Right Xiao"
- moved on the sheet: H3, H4

Commit message: feat: switch to new MCU, new journal
Parts:
- added C1, C2, C4, C7, C8: 100nF, symbol Device:C
- added C3, C6: 1uF, symbol Device:C
- added C5: 4.7uF, symbol Device:C
- added P3: USB_C_Plug_USB2.0, Connector_USB:USB_C_Receptacle_GCT_USB4105, symbol Connector:USB_C_Receptacle_USB2.0_14P
- added R1, R2: 5.1kO, symbol Device:R
- added R3: 10kO, symbol Device:R
- added S1: SKRPACE010, SKRPACE010:SW_SKRPACE010, symbol SKRPACE010:SKRPACE010
- added U2: SOT23, SOT23:SOT23, symbol SOT23:SOT23
- U1: footprint Package_QFP:LQFP-32_7x7mm_P0.8mm -> Package_DFN_QFN:WQFN-28-1EP_4x4mm_P0.4mm_EP2.7x2.7mm; symbol MCU_ST_STM32F0:STM32F042K6Tx -> MCU_WCH_RiscV:CH32X035G8U6
Connections:
- net COL10 is gone; now on net COL4: SW33.1, SW34.1, SW35.1, SW40.1
- net COL11 is gone; now on net COL5: SW37.1, SW38.1, SW39.1, SW51.1
- net COL6 is gone; now on net COL0: SW21.1, SW22.1, SW23.1
- net COL7 is gone; now on net COL1: SW24.1, SW25.1, SW26.1
- net COL8 is gone; now on net COL2: SW27.1, SW28.1, SW29.1
- net COL9 is gone; now on net COL3: SW30.1, SW31.1, SW32.1, SW36.1
- net COL0: now also P1.A6 (D+), P1.B6 (D+), P2.A6 (D+), P2.B6 (D+), U1.5 (PA0); no longer U1.6 (PA0)
- net COL1: now also P1.A7 (D-), P1.B7 (D-), P2.A7 (D-), P2.B7 (D-), U1.6 (PA1); no longer U1.7 (PA1)
- net COL2: now also P1.A2 (TX1+), P2.B11 (RX1+), U1.7 (PA2); no longer U1.8 (PA2)
- net COL3: now also P1.A3 (TX1-), P2.B10 (RX1-), U1.8 (PA3); no longer U1.9 (PA3)
- net COL4: now also P1.B2 (TX2+), P2.A11 (RX2+), U1.9 (PA4); no longer U1.10 (PA4)
- net COL5: now also P1.B3 (TX2-), P2.A10 (RX2-), U1.10 (PA5); no longer U1.11 (PA5)
- net ROW0: now also U1.13 (PB0); no longer U1.14 (PB0)
- net ROW1: now also U1.14 (PB3); no longer U1.15 (PB1)
- net ROW2: now also U1.15 (PB4); no longer U1.26 (PB3)
- net ROW3: now also U1.17 (PB6); no longer U1.27 (PB4)
- net ROW4: now also P1.B11 (RX1+), P2.A2 (TX1+), U1.18 (PB7); no longer U1.28 (PB5)
- net ROW5: now also P1.B10 (RX1-), P2.A3 (TX1-), U1.19 (PB8); no longer U1.29 (PB6)
- net ROW6: now also P1.A11 (RX2+), P2.B2 (TX2+), U1.20 (PB9); no longer U1.30 (PB7)
- net ROW7: now also P1.A10 (RX2-), P2.B3 (TX2-), U1.21 (PB10); no longer U1.31 (PB8)
- net at U1.2 (VDD): now also C3.2
- net GND_L renamed GND
- net GND: now also U1.29 (GND), C4.1, C5.2, C6.2, C7.1, C8.2, P3.A1 (GND), P3.A12 (GND), P3.B1 (GND), P3.B12 (GND), P3.SH (SHIELD), R1.2, R2.2, R3.1, U2.2 (P$2)
- new net: C2.2, C3.1
- new net: P3.A5 (CC1), R1.1
- new net: C7.2, R3.2, S1.1
- new net: P3.B5 (CC2), R2.1
- new net +3.3V: C1.1, C2.1, C4.2, S1.4, U2.1 (P$1)
- new net +3V3: C5.1
- new net DATA0: P3.A7 (D-), P3.B7 (D-), U1.26 (PC11/PC16/UDM)
- new net DATA1: P3.A6 (D+), P3.B6 (D+), U1.27 (PC10/PC17/UDP)
- new net LDO: C6.1, P3.A4 (VBUS), P3.A9 (VBUS), P3.B4 (VBUS), P3.B9 (VBUS), U2.3 (P$3)
- no-connect marks 0 -> 12
Other:
- note added: "Bulk Cap"
- note added: "Data Connection"
- note added: "Voltage Regulation"
- moved on the sheet: H3, H4

Commit message: feat: finish schematic, new journal entry
Parts:
- removed C1, C4, C7, C8: 100nF, symbol Device:C
- removed C3, C6: 1uF, symbol Device:C
- removed U2: SOT23, SOT23:SOT23, symbol SOT23:SOT23
- added TP1, TP2, TP3, TP4: TestPoint, TestPoint:TestPoint_Pad_D1.0mm, symbol Connector:TestPoint
- C2: footprint (none) -> Capacitor_SMD:C_0603_1608Metric
- C5: footprint (none) -> Capacitor_SMD:C_0805_2012Metric
- P1, P2: footprint Connector_USB:USB_C_Receptacle_GCT_USB4105 -> Connector_USB:USB_C_Receptacle_Molex_105450-0101
- P3: footprint Connector_USB:USB_C_Receptacle_GCT_USB4105 -> Connector_USB:USB_C_Receptacle_HRO_TYPE-C-31-M-12; symbol Connector:USB_C_Receptacle_USB2.0_14P -> Connector:USB_C_Receptacle_USB2.0_16P
- R1, R2: footprint (none) -> Resistor_SMD:R_0603_1608Metric
- R3: value 10kO -> 1k; footprint (none) -> Resistor_SMD:R_0603_1608Metric
- U1: value XIAO-RP2040-DIP -> CH32X035DS0
Connections:
- net +3.3V is gone; now on net +5V: C2.1, S1.4
- net +3V3 is gone; now on net +5V: C5.1
- net GND_R is gone; now on net GND: P2.A1 (GND), P2.A12 (GND), P2.B1 (GND), P2.B12 (GND), P2.SH (SHIELD)
- net LDO is gone; now on net +5V: P3.A4 (VBUS), P3.A9 (VBUS), P3.B4 (VBUS), P3.B9 (VBUS)
- net DATA1: now also R3.1
- net GND: now also C2.2, R3.2, S1.1, TP4.1; no longer R3.1
- net +5V: now reaches U1.2 (VDD)
- net +5V: now also TP3.1
- net at U1.24 (PC19/DCK): now also TP1.1
- net at U1.25 (PC18/DIO): now also TP2.1
- no-connect marks 12 -> 23
Other:
- note removed: "Voltage Regulation"
- moved on the sheet: C2, C5, H1, H2, R1, R2, S1

Commit message: feat: alomst finish new PCB routing
Parts:
- removed S1: SKRPACE010, SKRPACE010:SW_SKRPACE010, symbol SKRPACE010:SKRPACE010
- added SW41: SW_Push, Jumper:SolderJumper-2_P1.3mm_Open_Pad1.0x1.5mm, symbol Jumper:SolderJumper_2_Open
Connections:
- net +5V: now also SW41.2 (B)
- net GND: no longer R3.2
- new net: R3.2, SW41.1 (A)
- no-connect marks 23 -> 21
Other:
- moved on the sheet: R3

Commit message: feat: new journal, rename project, finish PCB
Other:
- note added: "Computer Connection"
- note removed: "Data Connection"
Changed lines of the file:
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@@
 	(text "Left MCU"
 		(exclude_from_sim no)
-		(at 20.828 108.712 0)
+		(at 21.082 108.966 0)
 		(effects
 			(font
@@
 		)
 	)
-	(text "Data Connection"
+	(text "Computer Connection"
 		(exclude_from_sim no)
 		(at 83.566 130.302 0)
@@
 	(text "Right Mounting"
 		(exclude_from_sim no)
-		(at 344.932 108.966 0)
+		(at 345.186 108.966 0)
 		(effects
 			(font
@@
 		(in_pos_files yes)
 		(dnp no)
-		(fields_autoplaced yes)
 		(property "Reference" "R3"
-			(at 64.77 121.9199 0)
+			(at 64.008 121.92 0)
 			(show_name no)
 			(do_not_autoplace no)
@@
 		)
 		(property "Value" "1k"
-			(at 64.77 124.4599 0)
+			(at 64.008 124.46 0)
 			(show_name no)
 			(do_not_autoplace no)
