File: kicad/snowlayer.kicad_pcb (KiCad board)
At the start: 2 copper layers, 270.5 x 89 mm, 103 parts, among them P1 USB_C_Plug_USB2.0, P2 USB_C_Plug_USB2.0, P3 USB_C_Plug_USB2.0, SW1 SW_Push, SW10 SW_Push, SW11 SW_Push, SW12 SW_Push, SW13 SW_Push, SW14 SW_Push, SW15 SW_Push, SW16 SW_Push, SW17 SW_Push, SW18 SW_Push, SW19 SW_Push, SW2 SW_Push, SW20 SW_Push, SW21 SW_Push, SW22 SW_Push, SW23 SW_Push, SW24 SW_Push, SW25 SW_Push, SW26 SW_Push, SW27 SW_Push, SW28 SW_Push, SW29 SW_Push, SW3 SW_Push, SW30 SW_Push, SW31 SW_Push, SW32 SW_Push, SW33 SW_Push, SW34 SW_Push, SW35 SW_Push, SW36 SW_Push, SW37 SW_Push, SW38 SW_Push, SW39 SW_Push, SW4 SW_Push, SW40 SW_Push, SW41 SW_Push, SW5 SW_Push, SW50 SW_Push, SW51 SW_Push, SW6 SW_Push, SW7 SW_Push, SW8 SW_Push, SW9 SW_Push, U1 CH32X035DS0

Commit message: feat: finish BOM, change out diodes + major rerouting, new journal entry
Parts:
- D1, D10, D11, D12, D13, D14, D15, D16, D17, D18, D19, D2, D20, D21, D22, D23, D24, D25, D26, D27, D28, D29, D3, D30, D31, D32, D33, D34, D35, D36, D37, D38, D39, D4, D40, D5, D50, D51, D6, D7, D8, D9: footprint Diode_SMD:D_SMA-SMB_Universal_Handsoldering -> Diode_SMD:D_SOD-123
- R3: value 1k -> 1kO
- moved D16 1.00 mm to (100.0, 141.0)
Routing:
- net /ROW5: track 150.5 -> 152.0 mm
- net Net-(D16-A): track 4.81 -> 3.49 mm
- net /ROW0: track 150.2 -> 151.3 mm
- net /ROW4: track 167.2 -> 168.2 mm
- net /ROW2: track 134.3 -> 133.6 mm
- net /ROW7: track 83.3 -> 84.0 mm
- net /ROW1: track 132.7 -> 132.2 mm
- net Net-(D9-A): track 4.10 -> 3.58 mm
- net Net-(D8-A): track 4.10 -> 3.58 mm
- net Net-(D7-A): track 4.10 -> 3.58 mm
- net Net-(D37-A): track 3.93 -> 3.41 mm
- net Net-(D35-A): track 5.00 -> 4.48 mm
- net Net-(D34-A): track 5.00 -> 4.48 mm
- net Net-(D33-A): track 5.00 -> 4.48 mm
- net Net-(D26-A): track 5.00 -> 4.48 mm
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
Commit message: feat: new journal, redo board outline
Parts:
- moved R3 10.4 mm to (120.9, 84.9)
- moved H4 5.81 mm to (244.9, 72.3)
- moved SW41 5.48 mm to (123.0, 84.9)
- moved H3 3.35 mm to (47.0, 70.8)
- moved P2 2.89 mm to (157.8, 115.5)
- moved H2 2.75 mm to (81.8, 125.5)
- moved D40 1.99 mm to (178.2, 143.8)
- moved D36 1.99 mm to (197.2, 140.8)
- moved D51 1.89 mm to (159.2, 138.4)
- moved SW36 1.54 mm to (197.2, 132.6)
- moved D39 1.51 mm to (273.2, 127.7)
- moved D33 1.50 mm to (254.2, 88.8)
- moved D34 1.50 mm to (254.3, 107.8)
- moved SW40 1.49 mm to (178.2, 135.7)
- moved SW51 1.45 mm to (159.1, 130.3)
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Routing:
- net /ROW7: track 84.0 -> 91.2 mm
- net Net-(D40-A): track 3.58 -> 0.00 mm
- net Net-(D36-A): track 3.58 -> 0.00 mm
- net GND: vias 21 -> 20
Other:
- board size 270.5 x 89 mm -> 268.1 x 87 mm

Commit message: feat: sync routing and new pcb design
Parts:
- moved C5 6.32 mm to (123.0, 104.0)
- moved G*** 5.37 mm to (224.3, 122.6)
- moved D25 4.05 mm to (193.4, 98.3)
- moved D37 3.95 mm to (269.6, 89.5)
- moved D31 3.92 mm to (231.5, 101.7)
- moved D51 3.90 mm to (155.3, 138.5)
- moved D40 3.90 mm to (174.3, 143.8)
- moved D23 3.86 mm to (174.3, 121.6)
- moved D36 3.81 mm to (193.4, 140.7)
- moved D22 3.81 mm to (174.3, 102.6)
- moved D21 3.80 mm to (174.4, 83.5)
- moved H1 3.80 mm to (205.9, 127.5)
- moved SW21 3.80 mm to (174.4, 75.4)
- moved SW22 3.80 mm to (174.3, 94.4)
- moved SW23 3.80 mm to (174.3, 113.5)
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Routing:
- net +5V: track 112.1 -> 22.1 mm
- net Net-(U1-PC19/DCK): track 78.1 -> 31.8 mm, vias 2 -> 0
- net Net-(U1-PC18/DIO): track 66.6 -> 28.0 mm, vias 2 -> 0
- net /DATA0: track 22.9 -> 0.00 mm
- net /COL5: track 301.4 -> 280.5 mm
- net /ROW1: track 132.2 -> 112.8 mm, vias 2 -> 1
- net /ROW0: track 151.3 -> 132.1 mm, vias 2 -> 1
- net /DATA1: track 39.6 -> 21.7 mm, vias 3 -> 0
- net /ROW2: track 133.6 -> 120.1 mm
- net Net-(P3-CC1): track 13.3 -> 1.10 mm, vias 2 -> 0
- net /COL4: track 332.0 -> 322.3 mm, vias 3 -> 2
- net /ROW3: track 79.5 -> 71.2 mm
- net GND: track 31.9 -> 39.6 mm, vias 20 -> 14
- net /COL3: track 321.8 -> 314.3 mm, vias 3 -> 2
- net Net-(P3-CC2): track 7.40 -> 0.00 mm
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Other:
- board size 268.1 x 87 mm -> 261.8 x 100.4 mm

Commit message: feat: new journal, better components
Parts:
- removed P1, P2: USB_C_Plug_USB2.0, Connector_USB:USB_C_Receptacle_Molex_105450-0101
- added USB1: TYPEC-24PIN_C53207800, snowlayer:USB-C-SMD_TYPE-C-24P-QT, F.Cu at (136.0, 116.5)
- added USB2: TYPEC-24PIN_C53207800, snowlayer:USB-C-SMD_TYPE-C-24P-QT, F.Cu at (156.2, 116.5)
- moved P3 1.80 mm to (139.0, 103.5)
Routing:
- net GND: track 39.6 -> 263.3 mm, vias 14 -> 8
- net /ROW4: track 163.2 -> 0.00 mm, vias 1 -> 0
- net /ROW6: track 146.5 -> 0.00 mm, vias 3 -> 0
- net /ROW5: track 146.0 -> 0.00 mm, vias 1 -> 0
- net /COL4: track 322.3 -> 211.1 mm, vias 2 -> 0
- net /COL2: track 274.5 -> 171.9 mm, vias 2 -> 0
- net /COL3: track 314.3 -> 218.4 mm, vias 2 -> 0
- net /ROW7: track 90.3 -> 0.00 mm, vias 3 -> 0
- net /COL5: track 280.5 -> 191.8 mm, vias 7 -> 0
- net /COL1: track 276.0 -> 189.5 mm, vias 5 -> 0
- net /COL0: track 271.8 -> 199.0 mm, vias 2 -> 0
- net /ROW0: track 132.1 -> 93.3 mm, vias 1 -> 0
- net /DATA1: track 21.7 -> 0.00 mm
- net /ROW1: track 112.8 -> 91.6 mm, vias 1 -> 0
- net /ROW3: track 71.2 -> 51.0 mm
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Other:
- board text removed: "P2"

Commit message: chore: upd readme
Parts:
- moved U1 4.49 mm to (128.2, 112.3), turned to -90 degrees
- moved R2 3.81 mm to (130.2, 105.0), turned to 180 degrees
- moved C5 3.69 mm to (126.5, 102.8), turned to 180 degrees
- moved R1 3.25 mm to (130.2, 103.3), turned to 180 degrees
- moved P3 2.99 mm to (137.3, 106.0)
- moved SW40 2.58 mm to (171.8, 135.5)
- moved D40 2.57 mm to (171.8, 143.6)
- moved SW51 2.57 mm to (152.7, 130.3)
- moved D51 2.57 mm to (152.7, 138.5)
- moved D33 2.56 mm to (248.0, 88.7)
- moved D34 2.56 mm to (248.0, 107.7)
- moved D35 2.56 mm to (248.0, 126.8)
- moved SW33 2.56 mm to (248.0, 80.5)
- moved SW34 2.56 mm to (248.0, 99.5)
- moved SW35 2.56 mm to (248.0, 118.6)
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Routing:
- net GND: track 263.3 -> 0.00 mm
- net /COL3: track 218.4 -> 0.00 mm
- net /COL4: track 211.1 -> 0.00 mm
- net /COL0: track 199.0 -> 0.00 mm
- net /COL5: track 191.8 -> 0.00 mm
- net /COL1: track 189.5 -> 0.00 mm
- net /COL2: track 171.9 -> 0.00 mm
- net /ROW2: track 107.1 -> 0.00 mm
- net /ROW0: track 93.3 -> 0.00 mm
- net /ROW1: track 91.6 -> 0.00 mm
- net /ROW3: track 51.0 -> 0.00 mm
- net Net-(U1-PC19/DCK): track 21.2 -> 0.00 mm
- net Net-(U1-PC18/DIO): track 20.8 -> 0.00 mm
- net /DATA1: track 0.00 -> 15.6 mm
- net +5V: track 22.1 -> 6.58 mm
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Other:
- board size 261.8 x 100.4 mm -> 259.2 x 84.1 mm

Commit message: feat: new journal, finish layout
Parts:
- moved H3 80.0 mm to (107.7, 123.0)
- moved H2 61.6 mm to (31.5, 90.0)
- moved H4 25.9 mm to (257.5, 90.0)
- moved H1 24.8 mm to (181.3, 123.0)
- moved G*** 4.84 mm to (217.0, 121.8)
- moved SW3 0.90 mm to (21.9, 118.6)
- moved SW1 0.90 mm to (21.9, 80.5)
- moved SW2 0.90 mm to (21.9, 99.5)
- moved SW37 0.90 mm to (267.1, 80.5)
- moved SW38 0.90 mm to (267.1, 99.5)
- moved SW39 0.90 mm to (267.1, 118.6)
- moved D3 0.80 mm to (21.9, 126.8)
- moved D39 0.80 mm to (267.1, 126.8)
- moved D1 0.80 mm to (21.9, 88.8)
- moved D2 0.80 mm to (21.9, 107.8)
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Other:
- board size 259.2 x 84.1 mm -> 259.2 x 84.6 mm

Commit message: feat: new journal, update all file outputs, finish routing/case
Parts:
- moved TP1 61.2 mm to (125.7, 129.8)
- moved TP2 61.2 mm to (125.7, 132.8)
- moved TP3 61.2 mm to (125.7, 135.8)
- moved TP4 61.2 mm to (125.7, 126.8)
- moved R3 25.2 mm to (128.9, 108.7), turned to 180 degrees
- moved SW41 20.8 mm to (126.2, 105.4), turned to 90 degrees
- moved U1 5.89 mm to (127.3, 118.1), turned to 0 degrees
- moved R1 2.71 mm to (128.9, 105.7)
- moved R2 2.58 mm to (128.9, 107.2)
- moved C2 2.29 mm to (128.9, 104.2)
- moved P3 1.60 mm to (135.7, 105.7)
- moved C5 0.75 mm to (125.7, 102.8)
Connections:
- U1 pad 18: /ROW4 -> /ROW5
- U1 pad 19: /ROW5 -> /ROW4
- U1 pad 20: /ROW6 -> /ROW7
- U1 pad 21: /ROW7 -> /ROW6
- USB1 pad A10: /ROW6 -> /ROW7
- USB1 pad A11: /ROW7 -> /ROW6
- USB2 pad B2: /ROW7 -> /ROW6
- USB2 pad B3: /ROW6 -> /ROW7
Routing:
- net /COL3: track 0.00 -> 327.0 mm, vias 0 -> 4
- net /COL4: track 0.00 -> 323.8 mm, vias 0 -> 3
- net /COL5: track 0.00 -> 297.0 mm, vias 0 -> 3
- net /COL2: track 0.00 -> 283.1 mm, vias 0 -> 3
- net /COL1: track 0.00 -> 281.3 mm, vias 0 -> 5
- net /COL0: track 0.00 -> 279.4 mm, vias 0 -> 5
- net /ROW4: track 0.00 -> 163.4 mm
- net /ROW0: track 0.00 -> 160.3 mm
- net /ROW5: track 0.00 -> 145.6 mm
- net /ROW1: track 0.00 -> 138.0 mm
- net /ROW6: track 4.37 -> 131.7 mm
- net /ROW2: track 0.00 -> 123.2 mm
- net +5V: track 6.58 -> 77.0 mm, vias 0 -> 3
- net /ROW7: track 3.37 -> 70.2 mm
- net /ROW3: track 0.00 -> 66.4 mm
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Other:
- board size 259.2 x 84.6 mm -> 259.2 x 85.6 mm
